File: QRD1114-bar.brd (EAGLE design)
At the start: 66 x 22 mm, 18 parts

Commit message: QRD1114-bar - small change in the board for better manufacturing
Parts:
- LED: device led:SML0603 -> led:SML0805
- moved R3 1.00 mm to (61.5, 5.00)
- moved R4 1.00 mm to (58.5, 5.00)
- moved R5 1.00 mm to (48.5, 5.00)
- moved R6 1.00 mm to (51.5, 5.00)
- moved R7 1.00 mm to (41.5, 5.00)
- moved R8 1.00 mm to (38.5, 5.00)
- moved LED 0.28 mm to (50.1, 14.0)
Routing:
- net S4: track 17.0 -> 16.0 mm
- net S3: track 17.9 -> 16.9 mm
- net S2: track 26.9 -> 25.9 mm
- net N$5: track 4.15 -> 3.15 mm
- net N$4: track 4.15 -> 3.15 mm
- net N$1: track 4.15 -> 3.15 mm
- net GND: track 1.00 -> 1.95 mm
